File: Altimeter_DualDeploy_KX1/KX1_DualDeployAltimeter_v100.brd (EAGLE design)
At the start: 48.3 x 50.8 mm, 40 parts, among them J1 AVR_SPI_PRG_6NS, U1 ATMEGA328P, U2 BMP180, Y3 16MHz

Commit message: Updated board design. Added .gitignore to ignore CAM output files
Parts:
- removed CH1: CH1, SparkFun-Connectors:1X02_LONGPADS
- removed CH2, CH3: CH2, SparkFun-Connectors:1X02_LONGPADS
- removed JP2: M02PTH3, SparkFun-Connectors:1X02_LONGPADS
- removed U$2: DIODE-ZENER-BZT52, SparkFun-DiscreteSemi:SOD-323
- added APOGEE_CHARGE: CH1, SparkFun-Connectors:1X02_LONGPADS
- added ARM_SWITCH, MAINS_CHARGE: CH2, SparkFun-Connectors:1X02_LONGPADS
- added C5, C6: 0.1uF, SparkFun-Capacitors:0603-CAP
- added C7: 470pF, SparkFun-Capacitors:0603-CAP
- added C8: 2.2uF, SparkFun-Capacitors:0603-CAP
- added PWR_IN: 3.6-16V, SparkFun-Connectors:1X02_LONGPADS
- added Z3: 3.3V, SparkFun-DiscreteSemi:SOD-323
- C4: value 0.1uF -> 1uF
- R11: value 1K -> 300
- R13, R8: value 10K -> 1K
- Z1, Z2: value DIODE-ZENER-BZT52 -> 3.3V
- moved JP5 29.9 mm to (41.9, 16.5)
- moved R13 26.4 mm to (17.8, 11.4), flipped to the bottom, turned to 270 degrees
- moved R12 25.1 mm to (20.3, 11.4), flipped to the bottom, turned to 90 degrees
- moved C1 21.0 mm to (15.2, 21.6), turned to 270 degrees
- moved R11 20.4 mm to (34.3, 24.1), turned to 180 degrees
- moved POWER 6.48 mm to (11.4, 22.9)
- moved U3 5.68 mm to (11.4, 15.2)
- moved C4 4.58 mm to (15.2, 10.2), turned to 0 degrees
- moved R8 2.54 mm to (6.35, 15.2), turned to 270 degrees
- moved Y3 1.47 mm to (18.5, 17.3), turned to 270 degrees
- moved C3 1.27 mm to (24.1, 17.8)
- renumbered U$1 to Z1, U$4 to Z2
Connections:
- removed net N$10: U$3.1
- net ARMED_CHECK: now also U1.1, Z3.1; no longer U$2.1, U1.19
- net DEPLOY1: now also APOGEE_CHARGE.2; no longer CH1.2
- net DEPLOY2: now also MAINS_CHARGE.2; no longer CH2.2, R13.2
- net GND: now also ARM_SWITCH.1, C5.2, C6.2, C7.2, C8.2, PWR_IN.2, Z3.2; no longer CH3.1, JP2.2, U$2.2
- net GND_ARMED: now also ARM_SWITCH.2, R13.2, U$3.1, U$3.3; no longer CH3.2
- net N$9: now also C7.1, U3.4; no longer U$3.3
- net VCC: now also C5.1, C6.1, C8.1; no longer R12.2
- net V_BATT: now also APOGEE_CHARGE.1, MAINS_CHARGE.1, PWR_IN.1, R12.2; no longer CH1.1, CH2.1, JP2.1
Routing:
- net V_BATT: track 11.4 -> 45.4 mm
- net GND_ARMED: track 0.00 -> 29.0 mm
- net ARMED_CHECK: track 0.00 -> 21.7 mm, vias 0 -> 3
- net GND: track 61.9 -> 82.5 mm, vias 6 -> 8
- net N$7: track 2.71 -> 12.4 mm
- net VCC: track 95.7 -> 104.0 mm, vias 4 -> 5
- net STATUS_LED: track 14.6 -> 6.41 mm
- net DEPLOY2: track 19.9 -> 27.5 mm
- net CHANNEL1: track 19.2 -> 23.9 mm
- net N$5: track 10.2 -> 5.66 mm
- net N$1: track 4.68 -> 8.56 mm
- net N$6: track 4.03 -> 7.83 mm
- net N$9: track 0.00 -> 3.05 mm
- net DEPLOY1: track 20.8 -> 22.8 mm
- net MISO: track 9.39 -> 8.05 mm
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Other:
- board text added: "( + )"
- board text added: "( - )"
- board text added: "+"
- board text added: "APOG"
- board text added: "ARM"
- board text added: "DTR"
- board text added: "MAINS"
- board text added: "RESET"
- board text added: "RXI"
- board text added: "STATUS"
- board text added: "TXO"
- board text added: "VCC"
- board text removed: "BAT"
- board text removed: "CH1"
- board text removed: "CH2"
