File: Altimeter_DualDeploy_KX1/KX1_DualDeployAltimeter_v100.sch (EAGLE design)
At the start: 40 parts, among them J1 AVR_SPI_PRG_6NS, U1 ATMEGA328P, U2 BMP180, Y3 16MHz

Commit message: Updated board design. Added .gitignore to ignore CAM output files
Parts:
- removed U$1, U$2, U$4: DIODE-ZENER-BZT52, SparkFun-DiscreteSemi:DIODE-ZENER-BZT52
- added C5, C6: 0.1uF, SparkFun-Capacitors:CAP0603-CAP
- added C7: 470pF, SparkFun-Capacitors:CAP0603-CAP
- added C8: 2.2uF, SparkFun-Capacitors:CAP0603-CAP
- added Z1, Z2, Z3: 3.3V, SparkFun-DiscreteSemi:DIODE-ZENER-BZT52
- C4: value 0.1uF -> 1uF
- PWR_IN: value M02PTH3 -> 3.6-16V
- R11: value 1K -> 300
- R13, R8: value 10K -> 1K
- renumbered CH1 to APOGEE_CHARGE, CH2 to MAINS_CHARGE, CH3 to ARM_SWITCH, JP2 to PWR_IN
Connections:
- removed net N$10: U$3.S@1
- net ARMED_CHECK: now also U1.PD3(INT1), Z3.C; no longer U$2.C, U1.ADC6
- net CONT_CHECK1: now also Z1.C; no longer U$1.C
- net CONT_CHECK2: now also Z2.C; no longer U$4.C
- net DEPLOY2: no longer R13.2
- net GND: now also C5.2, C6.2, C7.2, C8.2, Z1.A, Z2.A, Z3.A; no longer U$1.A, U$2.A, U$4.A
- net GND_ARMED: now also R13.2, U$3.S@1, U$3.S@3
- net N$9: now also C7.1, U3.BP; no longer U$3.S@3
- net VCC: now also C5.1, C6.1, C8.1; no longer R12.2
- net V_BATT: now also R12.2
Other:
- moved on the sheet: C2, POWER, R1, R3, R5, R8, S2, U2
